Commit message: v1.1

File: urdf/agv.urdf.xacro (robot description, xacro)
@@ -1,143 +1,27 @@
 <?xml version="1.0"?>
-<robot name="agv">
-  <!-- Base Link -->
+<robot xmlns:xacro="http://wiki.ros.org/xacro" name="agv">
+  <xacro:property name="wheel_radius" value="0.1"/>
+  <xacro:property name="wheel_separation" value="0.3"/>
   <link name="base_link">
-    <inertial>
-      <origin xyz="0 0 0" rpy="0 0 0"/>
-      <mass value="150"/>
-      <inertia ixx="10" ixy="0" ixz="0" iyy="10" iyz="0" izz="20"/>
-    </inertial>
-    <visual>
-      <origin xyz="0 0 0.25" rpy="0 0 0"/>
-      <geometry>
-        <box size="2.0 1.5 0.5"/>
-      </geometry>
-      <material name="blue">
-        <color rgba="0 0 1 1"/>
-      </material>
-    </visual>
-    <collision>
-      <origin xyz="0 0 0.25" rpy="0 0 0"/>
-      <geometry>
-        <box size="2.0 1.5 0.5"/>
-      </geometry>
-    </collision>
+    <inertial><mass value="10"/><origin xyz="0 0 0"/><inertia ixx="0.1" iyy="0.1" izz="0.1"/></inertial>
+    <visual><geometry><box size="0.5 0.3 0.1"/></geometry>
+    <material><color rgba="0 0 1 1"/></material></visual>
+    <collision><geometry><box size="0.5 0.3 0.1"/></geometry></collision>
   </link>
-  <!-- Front Left Wheel -->
-  <link name="front_left_wheel">
-    <inertial>
-      <origin xyz="0 0 0" rpy="0 0 0"/>
-      <mass value="10"/>
-      <inertia ixx="0.1" ixy="0" ixz="0" iyy="0.1" iyz="0" izz="0.1"/>
-    </inertial>
-    <visual>
-      <origin xyz="0 0 0" rpy="0 1.5708 0"/>
-      <geometry>
-        <cylinder length="0.2" radius="0.15"/>
-      </geometry>
-      <material name="black">
-        <color rgba="0 0 0 1"/>
-      </material>
-    </visual>
-    <collision>
-      <origin xyz="0 0 0" rpy="0 1.5708 0"/>
-      <geometry>
-        <cylinder length="0.2" radius="0.15"/>
-      </geometry>
-    </collision>
-  </link>
-  <!-- Front Right Wheel -->
-  <link name="front_right_wheel">
-    <inertial>
-      <origin xyz="0 0 0" rpy="0 0 0"/>
-      <mass value="10"/>
-      <inertia ixx="0.1" ixy="0" ixz="0" iyy="0.1" iyz="0" izz="0.1"/>
-    </inertial>
-    <visual>
-      <origin xyz="0 0 0" rpy="0 1.5708 0"/>
-      <geometry>
-        <cylinder length="0.2" radius="0.15"/>
-      </geometry>
-      <material name="black">
-        <color rgba="0 0 0 1"/>
-      </material>
-    </visual>
-    <collision>
-      <origin xyz="0 0 0" rpy="0 1.5708 0"/>
-      <geometry>
-        <cylinder length="0.2" radius="0.15"/>
-      </geometry>
-    </collision>
-  </link>
-  <!-- Rear Left Wheel -->
-  <link name="rear_left_wheel">
-    <inertial>
-      <origin xyz="0 0 0" rpy="0 0 0"/>
-      <mass value="10"/>
-      <inertia ixx="0.1" ixy="0" ixz="0" iyy="0.1" iyz="0" izz="0.1"/>
-    </inertial>
-    <visual>
-      <origin xyz="0 0 0" rpy="0 1.5708 0"/>
-      <geometry>
-        <cylinder length="0.2" radius="0.15"/>
-      </geometry>
-      <material name="black">
-        <color rgba="0 0 0 1"/>
-      </material>
-    </visual>
-    <collision>
-      <origin xyz="0 0 0" rpy="0 1.5708 0"/>
-      <geometry>
-        <cylinder length="0.2" radius="0.15"/>
-      </geometry>
-    </collision>
-  </link>
-  <!-- Rear Right Wheel -->
-  <link name="rear_right_wheel">
-    <inertial>
-      <origin xyz="0 0 0" rpy="0 0 0"/>
-      <mass value="10"/>
-      <inertia ixx="0.1" ixy="0" ixz="0" iyy="0.1" iyz="0" izz="0.1"/>
-    </inertial>
-    <visual>
-      <origin xyz="0 0 0" rpy="0 1.5708 0"/>
-      <geometry>
-        <cylinder length="0.2" radius="0.15"/>
-      </geometry>
-      <material name="black">
-        <color rgba="0 0 0 1"/>
-      </material>
-    </visual>
-    <collision>
-      <origin xyz="0 0 0" rpy="0 1.5708 0"/>
-      <geometry>
-        <cylinder length="0.2" radius="0.15"/>
-      </geometry>
-    </collision>
-  </link>
-  <!-- Joints Connecting Wheels to the Base -->
-  <joint name="front_left_wheel_joint" type="continuous">
-    <parent link="base_link"/>
-    <child link="front_left_wheel"/>
-    <origin xyz="0.9 0.75 0.2" rpy="0 0 0"/>
-    <axis xyz="0 1 0"/>
+  <link name="left_wheel_link"><visual><geometry><cylinder length="0.05" radius="${wheel_radius}"/></geometry></visual></link>
+  <link name="right_wheel_link"><visual><geometry><cylinder length="0.05" radius="${wheel_radius}"/></geometry></visual></link>
+  <joint name="left_wheel_joint" type="continuous">
+    <parent link="base_link"/><child link="left_wheel_link"/>
+    <origin xyz="0 ${wheel_separation/2} 0" rpy="0 1.5708 0"/><axis xyz="0 0 1"/>
   </joint>
-  <joint name="front_right_wheel_joint" type="continuous">
-    <parent link="base_link"/>
-    <child link="front_right_wheel"/>
-    <origin xyz="0.9 -0.75 0.2" rpy="0 0 0"/>
-    <axis xyz="0 1 0"/>
+  <joint name="right_wheel_joint" type="continuous">
+    <parent link="base_link"/><child link="right_wheel_link"/>
+    <origin xyz="0 -${wheel_separation/2} 0" rpy="0 1.5708 0"/><axis xyz="0 0 1"/>
   </joint>
-  <joint name="rear_left_wheel_joint" type="continuous">
-    <parent link="base_link"/>
-    <child link="rear_left_wheel"/>
-    <origin xyz="-0.9 0.75 0.2" rpy="0 0 0"/>
-    <axis xyz="0 1 0"/>
-  </joint>
-  <joint name="rear_right_wheel_joint" type="continuous">
-    <parent link="base_link"/>
-    <child link="rear_right_wheel"/>
-    <origin xyz="-0.9 -0.75 0.2" rpy="0 0 0"/>
-    <axis xyz="0 1 0"/>
-  </joint>
+  <gazebo><plugin name="diff_drive_controller" filename="libgazebo_ros_diff_drive.so">
+    <ros><namespace>/</namespace><remapping>cmd_vel:=cmd_vel</remapping></ros>
+    <updateRate>100.0</updateRate>
+    <leftJoint>left_wheel_joint</leftJoint><rightJoint>right_wheel_joint</rightJoint>
+    <wheelSeparation>${wheel_separation}</wheelSeparation><wheelDiameter>${wheel_radius*2}</wheelDiameter>
+  </plugin></gazebo>
 </robot>

Commit message: v1.2

File: urdf/agv.urdf.xacro (robot description, xacro)
@@ -4,24 +4,45 @@
   <xacro:property name="wheel_separation" value="0.3"/>
   <link name="base_link">
-    <inertial><mass value="10"/><origin xyz="0 0 0"/><inertia ixx="0.1" iyy="0.1" izz="0.1"/></inertial>
-    <visual><geometry><box size="0.5 0.3 0.1"/></geometry>
-    <material><color rgba="0 0 1 1"/></material></visual>
-    <collision><geometry><box size="0.5 0.3 0.1"/></geometry></collision>
+    <inertial>
+      <mass value="10"/>
+      <origin xyz="0 0 0"/>
+      <inertia ixx="0.1" iyy="0.1" izz="0.1"/>
+    </inertial>
+    <visual>
+      <geometry><box size="0.5 0.3 0.1"/></geometry>
+      <material><color rgba="0 0 1 1"/></material>
+    </visual>
+    <collision>
+      <geometry><box size="0.5 0.3 0.1"/></geometry>
+    </collision>
   </link>
-  <link name="left_wheel_link"><visual><geometry><cylinder length="0.05" radius="${wheel_radius}"/></geometry></visual></link>
-  <link name="right_wheel_link"><visual><geometry><cylinder length="0.05" radius="${wheel_radius}"/></geometry></visual></link>
+  <link name="left_wheel_link">
+    <visual><geometry><cylinder length="0.05" radius="${wheel_radius}"/></geometry></visual>
+  </link>
+  <link name="right_wheel_link">
+    <visual><geometry><cylinder length="0.05" radius="${wheel_radius}"/></geometry></visual>
+  </link>
   <joint name="left_wheel_joint" type="continuous">
     <parent link="base_link"/><child link="left_wheel_link"/>
-    <origin xyz="0 ${wheel_separation/2} 0" rpy="0 1.5708 0"/><axis xyz="0 0 1"/>
+    <origin xyz="0 ${wheel_separation/2} 0" rpy="0 1.5708 0"/>
+    <axis xyz="0 0 1"/>
   </joint>
   <joint name="right_wheel_joint" type="continuous">
     <parent link="base_link"/><child link="right_wheel_link"/>
-    <origin xyz="0 -${wheel_separation/2} 0" rpy="0 1.5708 0"/><axis xyz="0 0 1"/>
+    <origin xyz="0 -${wheel_separation/2} 0" rpy="0 1.5708 0"/>
+    <axis xyz="0 0 1"/>
   </joint>
-  <gazebo><plugin name="diff_drive_controller" filename="libgazebo_ros_diff_drive.so">
-    <ros><namespace>/</namespace><remapping>cmd_vel:=cmd_vel</remapping></ros>
-    <updateRate>100.0</updateRate>
-    <leftJoint>left_wheel_joint</leftJoint><rightJoint>right_wheel_joint</rightJoint>
-    <wheelSeparation>${wheel_separation}</wheelSeparation><wheelDiameter>${wheel_radius*2}</wheelDiameter>
-  </plugin></gazebo>
+  <gazebo>
+    <plugin name="diff_drive_controller" filename="libgazebo_ros_diff_drive.so">
+      <ros>
+        <namespace>/</namespace>
+        <remapping>cmd_vel:=cmd_vel</remapping>
+      </ros>
+      <updateRate>100.0</updateRate>
+      <leftJoint>left_wheel_joint</leftJoint>
+      <rightJoint>right_wheel_joint</rightJoint>
+      <wheelSeparation>${wheel_separation}</wheelSeparation>
+      <wheelDiameter>${wheel_radius*2}</wheelDiameter>
+    </plugin>
+  </gazebo>
 </robot>
